Commit message: upd README, ex03 robot description, add ex05

File: task5/ex03/ros2_ws/src/robot_description/urdf/robot.urdf.xacro (robot description, xacro)
@@ -1,10 +1,12 @@
-<?xml version="1.0" ?>
+<?xml version="1.0"?>
 <robot name='robot' xmlns:xacro="http://ros.org/wiki/xacro">
     <xacro:include filename="$(find robot_description)/urdf/gazebo.urdf.xacro" />
-    <!--xacro:include filename="$(find robot_description)/urdf/lidar.urdf.xacro" /-->
-    <!--xacro:include filename="$(find robot_description)/urdf/depth.urdf.xacro" /-->
-    <xacro:property name="chassis_length" value="0.335"/>
-    <xacro:property name="chassis_width" value="0.265"/>
-    <xacro:property name="chassis_height" value="0.138"/>
+    <!--xacro:include
+    filename="$(find robot_description)/urdf/lidar.urdf.xacro" /-->
+    <!--xacro:include
+    filename="$(find robot_description)/urdf/depth.urdf.xacro" /-->
+    <xacro:property name="chassis_length" value="0.335" />
+    <xacro:property name="chassis_width" value="0.265" />
+    <xacro:property name="chassis_height" value="0.138" />
     <xacro:property name="wheel_radius" value="0.033"/>
     <xacro:property name="wheel_thickness" value="0.026"/>
@@ -13,14 +15,26 @@
     <xacro:property name="wheel_offset_y" value="0.1485"/>
     <xacro:property name="wheel_offset_z" value="0.01"/>
-    <xacro:property name="caster_wheel_radius" value="0.01"/>
-    <xacro:property name="caster_wheel_mass" value="0.01"/>
-    <xacro:property name="caster_wheel_offset_x" value="0.075"/>
-    <xacro:property name="caster_wheel_offset_z" value="${wheel_offset_z - wheel_radius + caster_wheel_radius}"/>
-    <xacro:property name="mass" value="1.0"/>
+    <xacro:property name="caster_wheel_radius" value="0.03" />
+    <xacro:property name="caster_wheel_mass" value="0.01" />
+    <xacro:property name="caster_wheel_offset_x" value="0.075" />
+    <xacro:property name="caster_wheel_offset_z"
+    value="${wheel_offset_z - wheel_radius + caster_wheel_radius}" />
+    <xacro:property name="mass" value="1.0" />
+    <xacro:property name="antenna_radius" value="0.005"/>
+    <xacro:property name="antenna_length" value="0.15"/>
+    <xacro:property name="antenna_mass" value="0.01"/>
+    <xacro:property name="antenna_color" value="black"/>
+    <!-- Координаты установки антенн относительно корпуса -->
+    <xacro:property name="antenna1_x" value="${chassis_length * 0.8}"/>  <!-- Задняя часть корпуса -->
+    <xacro:property name="antenna1_y" value="${chassis_width * 0.3}"/>   <!-- Правая сторона -->
+    <xacro:property name="antenna1_z" value="${chassis_height}"/>        <!-- Верх корпуса -->
+    <xacro:property name="antenna2_x" value="${chassis_length * 0.8}"/>  <!-- Задняя часть корпуса -->
+    <xacro:property name="antenna2_y" value="${-chassis_width * 0.3}"/>  <!-- Левая сторона -->
+    <xacro:property name="antenna2_z" value="${chassis_height}"/>
     <material name="white">
-        <color rgba="1 1 1 1" />
+        <color rgba="0.71 0.75 1 1" />
     </material>
     <material name="orange">
-        <color rgba="1 0.3 0.1 1"/>
+        <color rgba="0.25 0.88 0.82 1" />  <!-- светло-бирюзовый / морская волна -->
     </material>
     <material name="blue">
@@ -28,8 +42,8 @@
     </material>
     <material name="black">
-        <color rgba="0 0 0 1"/>
+        <color rgba="0 0 0 1" />
     </material>
     <material name="red">
-        <color rgba="1 0 0 1"/>
+        <color rgba="1 0 0 1" />
     </material>
     <link name="base_link">
@@ -38,43 +52,45 @@
     </link>
     <joint name="base_footprint_joint" type="fixed">
-        <parent link="base_link"/>
-        <child link="base_footprint"/>
-        <origin xyz="0 0 -0.138" rpy="0 0 0"/>
+    <parent link="base_link" />
+    <child link="base_footprint" />
+    <origin xyz="0 0 -0.138" rpy="0 0 0" />
     </joint>
     <joint name="chassis_joint" type="fixed">
-        <parent link="base_link"/>
-        <child link="chassis"/>
-        <origin xyz="${-wheel_offset_x} 0 ${-wheel_offset_z}"/>
+    <parent link="base_link" />
+    <child link="chassis" />
+    <origin xyz="${-wheel_offset_x} 0 ${-wheel_offset_z}" />
     </joint>
     <link name='chassis'>
     <inertial>
-        <origin xyz="${chassis_length/2} 0 ${chassis_height/2}" rpy="0 0 0"/>
+        <origin xyz="${chassis_length/2} 0 ${chassis_height/2}" rpy="0 0 0" />
         <mass value="${mass}" />
-        <inertia ixx="${(1/12) * mass * (chassis_width*chassis_width+chassis_height*chassis_height)}" ixy="0.0" ixz="0.0"
-                 iyy="${(1/12) * mass * (chassis_length*chassis_length+chassis_height*chassis_height)}" iyz="0.0"
-                 izz="${(1/12) * mass * (chassis_length*chassis_length+chassis_width*chassis_width)}" />
-    </inertial>
-    <visual>
-        <origin xyz="${chassis_length/2} 0 ${chassis_height/2}"/>
-        <geometry>
-            <box size="${chassis_length} ${chassis_width} ${chassis_height}"/>
-        </geometry>
-        <material name="orange"/>
-    </visual>
-    <collision>
-        <origin xyz="${chassis_length/2} 0 ${chassis_height/2}"/>
-        <geometry>
-            <box size="${chassis_length} ${chassis_width} ${chassis_height}"/>
+        <inertia ixx="${(1/12) * mass * (chassis_width*chassis_width+chassis_height*chassis_height)}"
+        ixy="0.0" ixz="0.0"
+        iyy="${(1/12) * mass * (chassis_length*chassis_length+chassis_height*chassis_height)}"
+        iyz="0.0"
+        izz="${(1/12) * mass * (chassis_length*chassis_length+chassis_width*chassis_width)}" />
+    </inertial>
+    <visual>
+        <origin xyz="${chassis_length/2} 0 ${chassis_height/2}" />
+        <geometry>
+        <box size="${chassis_length} ${chassis_width} ${chassis_height}" />
+        </geometry>
+        <material name="orange" />
+    </visual>
+    <collision>
+        <origin xyz="${chassis_length/2} 0 ${chassis_height/2}" />
+        <geometry>
+        <box size="${chassis_length} ${chassis_width} ${chassis_height}" />
         </geometry>
     </collision>
     </link>
     <gazebo reference="chassis">
-        <material>Gazebo/Orange</material>
+    <material>Gazebo/SeaGreen</material>
     </gazebo>
     <joint name="left_wheel_joint" type="continuous">
-        <parent link="base_link"/>
-        <child link="left_wheel"/>
-        <origin xyz="0 ${wheel_offset_y} 0" rpy="-${pi/2} 0 0" />
-        <axis xyz="0 0 1"/>
+    <parent link="base_link" />
+    <child link="left_wheel" />
+    <origin xyz="0 ${wheel_offset_y} 0" rpy="-${pi/2} 0 0" />
+    <axis xyz="0 0 1" />
     </joint>
     <link name="left_wheel">
@@ -99,11 +115,11 @@
     </link>
     <gazebo reference="left_wheel">
-        <material>Gazebo/Blue</material>
+    <material>Gazebo/Blue</material>
     </gazebo>
     <joint name="right_wheel_joint" type="continuous">
-        <parent link="base_link"/>
-        <child link="right_wheel"/>
-        <origin xyz="0 ${-wheel_offset_y} 0" rpy="${pi/2} 0 0" />
-        <axis xyz="0 0 -1"/>
+    <parent link="base_link" />
+    <child link="right_wheel" />
+    <origin xyz="0 ${-wheel_offset_y} 0" rpy="${pi/2} 0 0" />
+    <axis xyz="0 0 -1" />
     </joint>
     <link name="right_wheel">
@@ -128,35 +144,128 @@
     </link>
     <gazebo reference="right_wheel">
-        <material>Gazebo/Blue</material>
+    <material>Gazebo/Blue</material>
     </gazebo>
     <joint name="caster_wheel_joint" type="fixed">
-        <parent link="chassis"/>
-        <child link="caster_wheel"/>
-        <origin xyz="${caster_wheel_offset_x} 0 ${caster_wheel_offset_z}"/>
+    <parent link="chassis" />
+    <child link="caster_wheel" />
+    <origin xyz="${caster_wheel_offset_x} 0 ${caster_wheel_offset_z}" />
     </joint>
     <link name="caster_wheel">
-        <visual>
-            <geometry>
-                <sphere radius="${caster_wheel_radius}"/>
-            </geometry>
-            <material name="white"/>
-        </visual>
-        <collision>
-            <geometry>
-                <sphere radius="${caster_wheel_radius}"/>
-            </geometry>
-        </collision>
-        <inertial>
-            <origin xyz="0 0 0" rpy="0 0 0"/>
-            <mass value="${caster_wheel_mass}" />
-            <inertia ixx="${(2/5) * caster_wheel_mass * (caster_wheel_radius*caster_wheel_radius)}" ixy="0.0" ixz="0.0"
-                     iyy="${(2/5) * caster_wheel_mass * (caster_wheel_radius*caster_wheel_radius)}" iyz="0.0"
-                     izz="${(2/5) * caster_wheel_mass * (caster_wheel_radius*caster_wheel_radius)}" />
-        </inertial>
+    <visual>
+        <geometry>
+        <sphere radius="${caster_wheel_radius}" />
+        </geometry>
+        <material name="white" />
+    </visual>
+    <collision>
+        <geometry>
+        <sphere radius="${caster_wheel_radius}" />
+        </geometry>
+    </collision>
+    <inertial>
+        <origin xyz="0 0 0" rpy="0 0 0" />
+        <mass value="${caster_wheel_mass}" />
+        <inertia ixx="${(2/5) * caster_wheel_mass * (caster_wheel_radius*caster_wheel_radius)}"
+        ixy="0.0" ixz="0.0"
+        iyy="${(2/5) * caster_wheel_mass * (caster_wheel_radius*caster_wheel_radius)}" iyz="0.0"
+        izz="${(2/5) * caster_wheel_mass * (caster_wheel_radius*caster_wheel_radius)}" />
+    </inertial>
     </link>
     <gazebo reference="caster_wheel">
-        <material>Gazebo/White</material>
-        <mu1 value="0.001"/>
-        <mu2 value="0.001"/>
-    </gazebo>
+    <material>Gazebo/White</material>
+    <mu1 value="0.001" />
+    <mu2 value="0.001" />
+    </gazebo>
+    <!-- Первая антенна (правая) -->
+    <link name="antenna_1">
+    <inertial>
+        <origin xyz="0 0 ${antenna_length/2}" rpy="0 0 0"/>
+        <mass value="${antenna_mass}" />
+        <inertia ixx="${(1/12) * antenna_mass * (3*antenna_radius*antenna_radius + antenna_length*antenna_length)}" ixy="0.0" ixz="0.0"
+                    iyy="${(1/12) * antenna_mass * (3*antenna_radius*antenna_radius + antenna_length*antenna_length)}" iyz="0.0"
+                    izz="${(1/2) * antenna_mass * antenna_radius*antenna_radius}" />
+    </inertial>
+    <visual>
+        <origin xyz="0 0 ${antenna_length/2}" rpy="0 0 0"/>
+        <geometry>
+            <cylinder radius="${antenna_radius}" length="${antenna_length}"/>
+        </geometry>
+        <material name="${antenna_color}"/>
+    </visual>
+    <collision>
+        <origin xyz="0 0 ${antenna_length/2}" rpy="0 0 0"/>
+        <geometry>
+            <cylinder radius="${antenna_radius}" length="${antenna_length}"/>
+        </geometry>
+    </collision>
+    </link>
+    <joint name="antenna_1_joint" type="fixed">
+    <parent link="chassis"/>  <!-- Привязка к корпусу -->
+    <child link="antenna_1"/>
+    <origin xyz="${antenna1_x} ${antenna1_y} ${antenna1_z}" rpy="0 0 0"/>
+    </joint>
+    <!-- Вторая антенна (левая) -->
+    <link name="antenna_2">
+    <inertial>
+        <origin xyz="0 0 ${antenna_length/2}" rpy="0 0 0"/>
+        <mass value="${antenna_mass}" />
+        <inertia ixx="${(1/12) * antenna_mass * (3*antenna_radius*antenna_radius + antenna_length*antenna_length)}" ixy="0.0" ixz="0.0"
+                    iyy="${(1/12) * antenna_mass * (3*antenna_radius*antenna_radius + antenna_length*antenna_length)}" iyz="0.0"
+                    izz="${(1/2) * antenna_mass * antenna_radius*antenna_radius}" />
+    </inertial>
+    <visual>
+        <origin xyz="0 0 ${antenna_length/2}" rpy="0 0 0"/>
+        <geometry>
+            <cylinder radius="${antenna_radius}" length="${antenna_length}"/>
+        </geometry>
+        <material name="${antenna_color}"/>
+    </visual>
+    <collision>
+        <origin xyz="0 0 ${antenna_length/2}" rpy="0 0 0"/>
+        <geometry>
+            <cylinder radius="${antenna_radius}" length="${antenna_length}"/>
+        </geometry>
+    </collision>
+    </link>
+    <joint name="antenna_2_joint" type="fixed">
+    <parent link="chassis"/>  <!-- Привязка к корпусу -->
+    <child link="antenna_2"/>
+    <origin xyz="${antenna2_x} ${antenna2_y} ${antenna2_z}" rpy="0 0 0"/>
+    </joint>
+    <!-- Gazebo материалы для антенн -->
+    <gazebo reference="antenna_1">
+    <material>Gazebo/Black</material>
+    </gazebo>
+    <gazebo reference="antenna_2">
+    <material>Gazebo/Black</material>
+    </gazebo>
+    <!-- Глаза на антеннах -->
+    <link name="eye_left">
+        <visual>
+        <origin xyz="0 0 0.15" rpy="0 0 0"/>
+        <geometry>
+            <sphere radius="0.03"/>
+        </geometry>
+        <material name="black"/>
+        </visual>
+    </link>
+    <joint name="eye_left_joint" type="fixed">
+        <parent link="antenna_1"/>
+        <child link="eye_left"/>
+        <origin xyz="0 0 0" rpy="0 0 0"/>
+    </joint>
+    <link name="eye_right">
+        <visual>
+        <origin xyz="0 0 0.15" rpy="0 0 0"/>
+        <geometry>
+            <sphere radius="0.03"/>
+        </geometry>
+        <material name="black"/>
+        </visual>
+    </link>
+    <joint name="eye_right_joint" type="fixed">
+        <parent link="antenna_2"/>
+        <child link="eye_right"/>
+        <origin xyz="0 0 0" rpy="0 0 0"/>
+    </joint>
 </robot>
