Commit message: upd task5/ex03

File: task5/ex03/ros2_ws/src/robot_description/urdf/V1_robot.urdf.xacro (robot description, xacro)
@@ -8,5 +8,5 @@
     <xacro:property name="chassis_length" value="0.335" />
     <xacro:property name="chassis_width" value="0.265" />
-    <xacro:property name="chassis_height" value="0.1" />
+    <xacro:property name="chassis_height" value="0.138" />
     <xacro:property name="wheel_radius" value="0.033"/>
     <xacro:property name="wheel_thickness" value="0.026"/>
@@ -35,7 +35,4 @@
         <color rgba="0.71 0.75 1 1" />
     </material>
-    <material name="rose">
-        <color rgba="0.812 0.604 0.659 1" />
-    </material>
     <material name="orange">
         <color rgba="0.25 0.88 0.82 1" />  <!-- светло-бирюзовый / морская волна -->
@@ -183,5 +180,5 @@
     <link name="antenna_1">
     <inertial>
-        <origin xyz="0.04 0 ${antenna_length/2}" rpy="0 0 0"/>
+        <origin xyz="0 0 ${antenna_length/2}" rpy="0 0 0"/>
         <mass value="${antenna_mass}" />
         <inertia ixx="${(1/12) * antenna_mass * (3*antenna_radius*antenna_radius + antenna_length*antenna_length)}" ixy="0.0" ixz="0.0"
@@ -190,5 +187,5 @@
     </inertial>
     <visual>
-        <origin xyz="0.04 0 ${antenna_length/2}" rpy="0 0 0"/>
+        <origin xyz="0 0 ${antenna_length/2}" rpy="0 0 0"/>
         <geometry>
             <cylinder radius="${antenna_radius}" length="${antenna_length}"/>
@@ -197,5 +194,5 @@
     </visual>
     <collision>
-        <origin xyz="0.04 0 ${antenna_length/2}" rpy="0 0 0"/>
+        <origin xyz="0 0 ${antenna_length/2}" rpy="0 0 0"/>
         <geometry>
             <cylinder radius="${antenna_radius}" length="${antenna_length}"/>
@@ -211,5 +208,5 @@
     <link name="antenna_2">
     <inertial>
-        <origin xyz="0.04 0 ${antenna_length/2}" rpy="0 0 0"/>
+        <origin xyz="0 0 ${antenna_length/2}" rpy="0 0 0"/>
         <mass value="${antenna_mass}" />
         <inertia ixx="${(1/12) * antenna_mass * (3*antenna_radius*antenna_radius + antenna_length*antenna_length)}" ixy="0.0" ixz="0.0"
@@ -218,5 +215,5 @@
     </inertial>
     <visual>
-        <origin xyz="0.04 0 ${antenna_length/2}" rpy="0 0 0"/>
+        <origin xyz="0 0 ${antenna_length/2}" rpy="0 0 0"/>
         <geometry>
             <cylinder radius="${antenna_radius}" length="${antenna_length}"/>
@@ -225,5 +222,5 @@
     </visual>
     <collision>
-        <origin xyz="0.04 0 ${antenna_length/2}" rpy="0 0 0"/>
+        <origin xyz="0 0 ${antenna_length/2}" rpy="0 0 0"/>
         <geometry>
             <cylinder radius="${antenna_radius}" length="${antenna_length}"/>
@@ -246,5 +243,5 @@
     <link name="eye_left">
         <visual>
-        <origin xyz="0.04 0 0.15" rpy="0 0 0"/>
+        <origin xyz="0 0 0.15" rpy="0 0 0"/>
         <geometry>
             <sphere radius="0.03"/>
@@ -260,5 +257,5 @@
     <link name="eye_right">
         <visual>
-        <origin xyz="0.04 0 0.15" rpy="0 0 0"/>
+        <origin xyz="0 0 0.15" rpy="0 0 0"/>
         <geometry>
             <sphere radius="0.03"/>
@@ -272,32 +269,3 @@
         <origin xyz="0 0 0" rpy="0 0 0"/>
     </joint>
-    <!-- Сфера сверху -->
-    <link name="body_sphere">
-      <visual>
-        <origin xyz="0.12 0 ${chassis_height + 0.1}" rpy="0 0 0"/>
-        <geometry>
-          <sphere radius="0.15"/>
-        </geometry>
-        <material name="rose"/>
-      </visual>
-      <collision>
-        <origin xyz="0.1 0 ${chassis_height+ 0.1}" rpy="0 0 0"/>
-        <geometry>
-          <sphere radius="0.15"/>
-        </geometry>
-      </collision>
-      <inertial>
-        <mass value="0.5"/>
-        <origin xyz="0.1 0 ${chassis_height + 0.1}" rpy="0 0 0"/>
-        <inertia ixx="0.02" ixy="0" ixz="0" iyy="0.02" iyz="0" izz="0.02"/>
-      </inertial>
-    </link>
-    <joint name="body_sphere_joint" type="fixed">
-        <parent link="chassis"/>
-        <child link="body_sphere"/>
-        <origin xyz="0 0 0" rpy="0 0 0"/>
-    </joint>
-    <gazebo reference="body_sphere">
-    <material>Gazebo/Rose</material>
-    </gazebo>
 </robot>
